File: Control.kicad_sch (KiCad schematic)
At the start: 8 parts, among them U3 STM32F411VCHx

Commit message: not adding this to source control months ago was one of the dumbest things i've ever done. and im not particularly risk-avers
Parts:
- BT1: value Coin Cell -> BU2032SM-JJ-GTR; footprint (none) -> Battery:BAT_BU2032SM-JJ-GTR; Datasheet_local (none) -> {KIPROJMOD]/datasheets/BU2030SM-JJ-GTR.pdf
- C8: value 100 nF -> 0.1µF; footprint (none) -> easyeda2kicad:C0402
Connections:
- net AUX_GPIO_PB5 renamed SCREEN_BRIGHTNESS_PWM
- net HMI/SCREEN_BRIGHTNESS renamed HMI/SD_DETECT
Other:
- sheet HMI ports: added SD_DETECT; removed none
- moved on the sheet: BT1
