File: HMI.kicad_sch (KiCad schematic)
At the start: 0 parts

Commit message: not adding this to source control months ago was one of the dumbest things i've ever done. and im not particularly risk-avers
Other:
- sheet SD ports: added Card Detect; removed none
Changed lines of the file:
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@@
+	(wire
+		(pts
+			(xy 121.92 86.36) (xy 134.62 86.36)
+		)
+		(stroke
+			(width 0)
+			(type default)
+		)
+	)
 	(wire
 		(pts
@@
 			)
 			(justify right)
+		)
+	)
+	(hierarchical_label "SD_DETECT"
+		(shape output)
+		(at 134.62 86.36 0)
+		(effects
+			(font
+				(size 1.27 1.27)
+			)
+			(justify left)
 		)
 	)
@@
 	)
 	(sheet
-		(at 88.9 86.36)
-		(size 33.02 12.7)
+		(at 88.9 83.058)
+		(size 33.02 16.002)
 		(exclude_from_sim no)
 		(in_bom yes)
@@
 		)
 		(property "Sheetname" "SD"
-			(at 88.9 85.598 0)
+			(at 88.9 82.296 0)
 			(effects
 				(font
@@
 		)
 		(property "Sheetfile" "sd_card.kicad_sch"
-			(at 88.9 101.5496 0)
+			(at 88.9 99.822 0)
 			(effects
 				(font
@@
 				)
 				(justify right)
+			)
+		)
+		(pin "Card Detect" output
+			(at 121.92 86.36 0)
+			(effects
+				(font
+					(size 1.27 1.27)
+				)
+				(justify right)
