File: aux_term.kicad_sch (KiCad schematic)
At the start: 2 parts, among them J11 AUX port

Commit message: not adding this to source control months ago was one of the dumbest things i've ever done. and im not particularly risk-avers
Parts:
- added C36: C, symbol Device:C
Connections:
- net Aux GPIO BP5 is gone; now on net Aux GPIO BP10: J11.5 (Pin_5)
- net +3V3: now also J11.10 (Pin_10), C36.1
- net AUX_UART_RX: now also J11.8 (Pin_8); no longer J11.9 (Pin_9)
- net AUX_UART_TX: now also J11.9 (Pin_9); no longer J11.10 (Pin_10)
- net AUX_USART_CK: now also J11.7 (Pin_7); no longer J11.8 (Pin_8)
- net Aux GPIO BP10: no longer J11.6 (Pin_6)
- net Aux GPIO BP11: now also J11.6 (Pin_6); no longer J11.7 (Pin_7)
- net GND: now also C36.2
