File: crystal.kicad_sch (KiCad schematic)
At the start: 3 parts, among them Y1 Crystal

Commit message: not adding this to source control months ago was one of the dumbest things i've ever done. and im not particularly risk-avers
Parts:
- C6, C7: footprint (none) -> easyeda2kicad:C0603
Changed lines of the file:
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@@
 			)
 		)
-		(property "Footprint" ""
+		(property "Footprint" "easyeda2kicad:C0603"
 			(at 191.4652 130.81 0)
 			(effects
@@
 			)
 		)
-		(property "Datasheet" "~"
+		(property "Datasheet" "https://www.lcsc.com/datasheet/C2170082.pdf?spm=wm.sxq.inf.ggs___wm.fly.bg.0.xh&lcsc_vid=FFUIUwFUT1YIXlRVTlZZAQUAFFMKAlIFQFVbX1RXRwUxVlNeRldfUlRXQFVeXjsOAxUeFF5JWBYZEEoKFBINSQcJGk4dAgUUFAk%3D"
 			(at 190.5 127 0)
 			(effects
@@
 			)
 		)
-		(property "Footprint" ""
+		(property "Footprint" "easyeda2kicad:C0603"
 			(at 168.6052 130.81 0)
 			(effects
@@
 			)
 		)
-		(property "Datasheet" "~"
+		(property "Datasheet" "https://www.lcsc.com/datasheet/C2170082.pdf?spm=wm.sxq.inf.ggs___wm.fly.bg.0.xh&lcsc_vid=FFUIUwFUT1YIXlRVTlZZAQUAFFMKAlIFQFVbX1RXRwUxVlNeRldfUlRXQFVeXjsOAxUeFF5JWBYZEEoKFBINSQcJGk4dAgUUFAk%3D"
 			(at 167.64 127 0)
 			(effects
